Commit message: feat(arm): 볼 잠금 URDF와 MoveIt 가상 검증 기록 추가

File: extreme-robot/ros2_ws/src/robot_arm_description/urdf/robot_arm.urdf (robot description, URDF)
Before this commit: robot robot_arm, 52 links, 51 joints
Links:
- removed link link_001
- removed link link_002
- removed link link_003
- removed link link_004
- removed link link_005
- removed link link_006
- removed link link_007
- removed link link_008
- removed link link_009
- removed link link_010
- removed link link_011
- removed link link_012
- removed link link_013
- removed link link_014
- removed link link_015
- removed link link_016
- removed link link_017
- removed link link_018
- removed link link_019
- removed link link_020
- removed link link_021
- removed link link_022
- removed link link_023
- removed link link_024
- removed link link_025
- removed link link_026
- removed link link_027
- removed link link_028
- removed link link_029
- removed link link_030
- removed link link_031
- removed link link_032
- removed link link_033
- removed link link_034
- removed link link_035
- removed link link_036
- removed link link_037
- removed link link_038
- removed link link_040
- removed link link_041
- removed link link_042
- removed link link_044
- removed link link_045
- removed link link_046
- removed link link_047
- removed link link_048
- removed link link_049
- removed link link_050
- removed link wrist_camera_link
- added link arm_axis1_motor, mass 0.165; collision mesh filename=package://robot_arm_description/meshes/ball_lock/arm_axis1_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 scale=0.001 0.001 0.001; visual mesh filename=package://robot_arm_description/meshes/ball_lock/arm_axis1_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 scale=0.001 0.001 0.001
- added link arm_link1, mass 1.58123; collision mesh filename=package://robot_arm_description/meshes/ball_lock/arm_link1.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 scale=0.001 0.001 0.001; visual mesh filename=package://robot_arm_description/meshes/ball_lock/arm_link1.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 scale=0.001 0.001 0.001
- added link arm_link2, mass 1.87434; collision mesh filename=package://robot_arm_description/meshes/ball_lock/arm_link2.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 scale=0.001 0.001 0.001; visual mesh filename=package://robot_arm_description/meshes/ball_lock/arm_link2.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 scale=0.001 0.001 0.001
- added link arm_link3, mass 1.05513; collision mesh filename=package://robot_arm_description/meshes/ball_lock/arm_link3.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 scale=0.001 0.001 0.001; visual mesh filename=package://robot_arm_description/meshes/ball_lock/arm_link3.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 scale=0.001 0.001 0.001
- added link arm_link4, mass 0.0100505; collision mesh filename=package://robot_arm_description/meshes/ball_lock/arm_link4.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 scale=0.001 0.001 0.001; visual mesh filename=package://robot_arm_description/meshes/ball_lock/arm_link4.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 scale=0.001 0.001 0.001
- added link arm_link5, mass 0.883874; collision mesh filename=package://robot_arm_description/meshes/ball_lock/arm_link5.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 scale=0.001 0.001 0.001; visual mesh filename=package://robot_arm_description/meshes/ball_lock/arm_link5.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 scale=0.001 0.001 0.001
- added link finger_lower, mass 0.124979; collision mesh filename=package://robot_arm_description/meshes/ball_lock/finger_low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 scale=0.001 0.001 0.001; visual mesh filename=package://robot_arm_description/meshes/ball_lock/finger_low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 scale=0.001 0.001 0.001
- added link finger_upper, mass 0.124995; collision mesh filename=package://robot_arm_description/meshes/ball_lock/finger_upp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 scale=0.001 0.001 0.001; visual mesh filename=package://robot_arm_description/meshes/ball_lock/finger_upp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 scale=0.001 0.001 0.001
- added link pinion_A, mass 0.0112643; collision mesh filename=package://robot_arm_description/meshes/ball_lock/pinion_A.s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 scale=0.001 0.001 0.001; visual mesh filename=package://robot_arm_description/meshes/ball_lock/pinion_A.s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 scale=0.001 0.001 0.001
- added link pinion_B, mass 0.0112643; collision mesh filename=package://robot_arm_description/meshes/ball_lock/pinion_B.s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 scale=0.001 0.001 0.001; visual mesh filename=package://robot_arm_description/meshes/ball_lock/pinion_B.s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 scale=0.001 0.001 0.001
- added link tool_link, mass 0.377085; collision mesh filename=package://robot_arm_description/meshes/ball_lock/tool_link.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 scale=0.001 0.001 0.001; visual mesh filename=package://robot_arm_description/meshes/ball_lock/tool_link.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 scale=0.001 0.001 0.001
- added link toolchanger_ball_1, mass 0.000332422; collision mesh filename=package://robot_arm_description/meshes/ball_lock/toolchange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 scale=0.001 0.001 0.001; visual mesh filename=package://robot_arm_description/meshes/ball_lock/toolchange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 scale=0.001 0.001 0.001
- added link toolchanger_ball_2, mass 0.000332422; collision mesh filename=package://robot_arm_description/meshes/ball_lock/toolchange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 scale=0.001 0.001 0.001; visual mesh filename=package://robot_arm_description/meshes/ball_lock/toolchange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 scale=0.001 0.001 0.001
- added link toolchanger_ball_3, mass 0.000332422; collision mesh filename=package://robot_arm_description/meshes/ball_lock/toolchange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 scale=0.001 0.001 0.001; visual mesh filename=package://robot_arm_description/meshes/ball_lock/toolchange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 scale=0.001 0.001 0.001
- added link toolchanger_ball_4, mass 0.000332422; collision mesh filename=package://robot_arm_description/meshes/ball_lock/toolchange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 scale=0.001 0.001 0.001; visual mesh filename=package://robot_arm_description/meshes/ball_lock/toolchange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 scale=0.001 0.001 0.001
- added link toolchanger_ball_5, mass 0.000332422; collision mesh filename=package://robot_arm_description/meshes/ball_lock/toolchange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 scale=0.001 0.001 0.001; visual mesh filename=package://robot_arm_description/meshes/ball_lock/toolchange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 scale=0.001 0.001 0.001
- added link toolchanger_ball_6, mass 0.000332422; collision mesh filename=package://robot_arm_description/meshes/ball_lock/toolchange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 scale=0.001 0.001 0.001; visual mesh filename=package://robot_arm_description/meshes/ball_lock/toolchange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 scale=0.001 0.001 0.001
- added link toolchanger_ball_7, mass 0.000332422; collision mesh filename=package://robot_arm_description/meshes/ball_lock/toolchange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 scale=0.001 0.001 0.001; visual mesh filename=package://robot_arm_description/meshes/ball_lock/toolchange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 scale=0.001 0.001 0.001
- added link toolchanger_ball_8, mass 0.000332422; collision mesh filename=package://robot_arm_description/meshes/ball_lock/toolchange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 scale=0.001 0.001 0.001; visual mesh filename=package://robot_arm_description/meshes/ball_lock/toolchange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 scale=0.001 0.001 0.001
- added link toolchanger_lock_rotor, mass 0.0102117; collision mesh filename=package://robot_arm_description/meshes/ball_lock/toolchange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 scale=0.001 0.001 0.001; visual mesh filename=package://robot_arm_description/meshes/ball_lock/toolchange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 scale=0.001 0.001 0.001
- link base_link: mass 0.0940875583823606 -> 0.527733; geometry collision mesh filename=package://robot_arm_description/meshes/ball_lock/base_link.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 scale=0.001 0.001 0.001; visual mesh filename=package://robot_arm_description/meshes/ball_lock/base_link.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 scale=0.001 0.001 0.001
- link link_043: mass 0.5057750603466008 -> None; geometry 
- link link_051: mass 0.009342052845410124 -> None; geometry 
Joints:
- removed joint fixed_joint_001
- removed joint fixed_joint_002
- removed joint fixed_joint_003
- removed joint fixed_joint_004
- removed joint fixed_joint_005
- removed joint fixed_joint_006
- removed joint fixed_joint_007
- removed joint fixed_joint_008
- removed joint fixed_joint_009
- removed joint fixed_joint_010
- removed joint fixed_joint_011
- removed joint fixed_joint_012
- removed joint fixed_joint_013
- removed joint fixed_joint_014
- removed joint fixed_joint_015
- removed joint fixed_joint_016
- removed joint fixed_joint_017
- removed joint fixed_joint_018
- removed joint fixed_joint_019
- removed joint fixed_joint_020
- removed joint fixed_joint_021
- removed joint fixed_joint_022
- removed joint fixed_joint_023
- removed joint fixed_joint_024
- removed joint fixed_joint_025
- removed joint fixed_joint_026
- removed joint fixed_joint_027
- removed joint fixed_joint_028
- removed joint fixed_joint_029
- removed joint fixed_joint_030
- removed joint fixed_joint_031
- removed joint fixed_joint_032
- removed joint fixed_joint_033
- removed joint fixed_joint_034
- removed joint fixed_joint_035
- removed joint fixed_joint_036
- removed joint fixed_joint_037
- removed joint fixed_joint_038
- removed joint fixed_joint_039
- removed joint fixed_joint_040
- removed joint fixed_joint_041
- removed joint fixed_joint_042
- added joint arm_axis1_motor_fixed: type fixed, parent base_link, child arm_axis1_motor, origin xyz=0 0 0 rpy=0 0 0
- added joint arm_link5_to_link_043: type fixed, parent arm_link5, child link_043, origin xyz=0 0 0 rpy=0 0 0
- added joint arm_link5_to_link_051: type fixed, parent arm_link5, child link_051, origin xyz=0 0 0 rpy=0 0 0
- added joint arm_tool_fixed: type fixed, parent arm_link4, child tool_link, origin xyz=0 -0.021625 0 rpy=0 0 0
- added joint lock_ball_1: type prismatic, parent arm_link5, child toolchanger_ball_1, origin xyz=0.0558026 0.0225931 -2.64069e-06 rpy=0 0 0, axis 0 -1 0, limit lower=0 upper=0.00259 effort=50 velocity=0.05
- added joint lock_ball_2: type prismatic, parent arm_link5, child toolchanger_ball_2, origin xyz=0.0558026 0.0159758 0.0159731 rpy=0 0 0, axis 0 -0.707107 -0.707107, limit lower=0 upper=0.00259 effort=50 velocity=0.05
- added joint lock_ball_3: type prismatic, parent arm_link5, child toolchanger_ball_3, origin xyz=0.0558026 7.72711e-16 0.0225905 rpy=0 0 0, axis 0 0 -1, limit lower=0 upper=0.00259 effort=50 velocity=0.05
- added joint lock_ball_4: type prismatic, parent arm_link5, child toolchanger_ball_4, origin xyz=0.0558026 -0.0159758 0.0159731 rpy=0 0 0, axis 0 0.707107 -0.707107, limit lower=0 upper=0.00259 effort=50 velocity=0.05
- added joint lock_ball_5: type prismatic, parent arm_link5, child toolchanger_ball_5, origin xyz=0.0558026 -0.0225931 -2.64069e-06 rpy=0 0 0, axis 0 1 0, limit lower=0 upper=0.00259 effort=50 velocity=0.05
- added joint lock_ball_6: type prismatic, parent arm_link5, child toolchanger_ball_6, origin xyz=0.0558026 -0.0159758 -0.0159784 rpy=0 0 0, axis 0 0.707107 0.707107, limit lower=0 upper=0.00259 effort=50 velocity=0.05
- added joint lock_ball_7: type prismatic, parent arm_link5, child toolchanger_ball_7, origin xyz=0.0558026 3.37512e-16 -0.0225958 rpy=0 0 0, axis 0 0 1, limit lower=0 upper=0.00259 effort=50 velocity=0.05
- added joint lock_ball_8: type prismatic, parent arm_link5, child toolchanger_ball_8, origin xyz=0.0558026 0.0159758 -0.0159784 rpy=0 0 0, axis 0 -0.707107 0.707107, limit lower=0 upper=0.00259 effort=50 velocity=0.05
- added joint toolchanger_lock_wheel: type revolute, parent arm_link5, child toolchanger_lock_rotor, origin xyz=0.0610526 1.12795e-15 -2.64069e-06 rpy=0 0 0, axis 1 0 0, limit lower=0 upper=0.392699 effort=10 velocity=2.0
- joint arm_joint_1: axis 0.0 0.0 1.0 -> 0 0 -1; child link_004 -> arm_link1; origin xyz=0.0 0.0 0.0465 rpy=0 0 0 -> xyz=0.1565 0 0.1321 rpy=0 0 0; parent link_002 -> arm_axis1_motor
- joint arm_joint_2: axis 1.0 0.0 0.0 -> 0 -1 0; child link_010 -> arm_link2; limit lower=0.0 upper=3.141593 effort=100 velocity=100 -> lower=-3.14159 upper=0 effort=10 velocity=2.0; origin xyz=0.0465 0.0 0.0 rpy=0 0 0 -> xyz=0.01021 0 0.0679 rpy=0 0 0; parent link_009 -> arm_link1
- joint arm_joint_3: axis -1.0 0.0 -0.0 -> 0 1 0; child link_022 -> arm_link3; limit lower=0.0 upper=3.141593 effort=100 velocity=100 -> lower=-3.14159 upper=0 effort=10 velocity=2.0; origin xyz=-0.0755 0.0 0.0 rpy=0 0 0 -> xyz=-0.293 0 0.06006 rpy=0 0 0; parent link_021 -> arm_link2
- joint arm_joint_4: axis -1.0 0.0 0.0 -> 0 1 0; child link_030 -> arm_link4; limit lower=-0.610865 upper=0.698132 effort=100 velocity=100 -> lower=-1.74533 upper=1.74533 effort=10 velocity=2.0; origin xyz=0.0001 -0.068917 0.0045 rpy=0 0 0 -> xyz=0.258002 0.021875 0.0600043 rpy=0 0 0; parent link_028 -> arm_link3
- joint arm_joint_5: axis 0.0 -1.0 0.0 -> 1 0 0; child link_040 -> arm_link5; limit (none) -> lower=-3.14159 upper=3.14159 effort=10 velocity=2.0; origin xyz=0.0309 0.001644 -0.00525 rpy=0 0 0 -> xyz=0.103998 -1.32815e-17 4.28408e-06 rpy=0 0 0; parent link_037 -> tool_link; type continuous -> revolute
- joint gripper_left_pinion_joint: axis 0.0 -1.0 -0.0 -> 1 0 0; child link_050 -> pinion_A; limit lower=0.0 upper=1.9444444444444444 effort=100 velocity=100 -> lower=-1.67901 upper=2.51443 effort=10 velocity=2.0; origin xyz=0.0 -0.006 0.0 rpy=0 0 0 -> xyz=0.11155 0.0200001 4.70805e-07 rpy=0 0 0; parent link_048 -> arm_link5
- joint gripper_left_rack_joint: axis 1.0 -0.0 -0.0 -> 0 1 0; child link_046 -> finger_lower; limit lower=-0.035 upper=0.0 effort=100 velocity=100 -> lower=-0.0452597 upper=0.0302221 effort=50 velocity=0.05; mimic joint=gripper_left_pinion_joint multiplier=-0.018 offset=0.0 -> (none); origin xyz=-0.098787 -0.259411 0.161136 rpy=0 0 0 -> xyz=0.11155 0.0946431 0.0172465 rpy=0 0 0; parent link_043 -> arm_link5
- joint gripper_right_pinion_joint: axis -0.0 -1.0 -0.0 -> 1 0 0; child link_051 -> pinion_B; limit lower=0.0 upper=1.9444444444444444 effort=100 velocity=100 -> lower=-1.67901 upper=2.51443 effort=10 velocity=2.0; mimic joint=gripper_left_pinion_joint multiplier=1.0 offset=0.0 -> (none); origin xyz=0.0 -0.004 0.0 rpy=0 0 0 -> xyz=0.11155 -0.02 -1.11022e-16 rpy=0 0 0; parent link_049 -> arm_link5
- joint gripper_right_rack_joint: axis -1.0 0.0 0.0 -> 0 1 0; child link_047 -> finger_upper; limit lower=-0.035 upper=0.0 effort=100 velocity=100 -> lower=-0.0302221 upper=0.0452597 effort=50 velocity=0.05; mimic joint=gripper_left_pinion_joint multiplier=-0.018 offset=0.0 -> (none); origin xyz=-0.109737 -0.047 -0.052497 rpy=0 0 0 -> xyz=0.11155 -0.0945769 -0.0172465 rpy=0 0 0; parent link_043 -> arm_link5

File: extreme-robot/ros2_ws/src/robot_arm_description/urdf/robot_arm.urdf.xacro (robot description, xacro)
@@ -1,11 +1,6 @@
 <?xml version="1.0"?>
-<!-- 메인 xacro: robot_arm.urdf(팔 5축 + link_051 아래 ee_description fixed base)를 include.
-     robot_arm.urdf는 <robot> 태그를 가진 완성 URDF지만,
-     xacro:include는 루트 태그 이름과 무관하게 자식 엘리먼트를 그대로 이 파일의 <robot>에 이어붙임.
-     이전엔 여기서 xacro:arg gripper로 그리퍼 모듈(urdf/grippers/*.xacro)을 골라 wrist_to_gripper
-     fixed joint로 짜맞췄으나, 서로 다른 CAD export(팔/그리퍼 각각 다른 리비전)의 좌표계를 맞추는
-     시도가 반복적으로 어긋나 폐기(2026-07-15, 사용자 결정) — robot_arm.urdf 헤더 주석 참고.
-     ee_description.zip에는 joint/TCP가 전혀 없다. 따라서 MoveIt joint를 만들지 않으며,
-     별도 actuator는 하드웨어 사양이 주어질 때까지 fail-closed로 둔다. -->
+<!-- dual_motor_gripper는 2026-10-14 볼 잠금 CAD 모델을 사용한다.
+     single_motor_gripper는 별도 기존 모델을 유지한다.
+     잠금 로터/볼 상태는 독립 관절이며 기구 연동식은 아직 제공되지 않았다. -->
 <robot name="robot_arm" xmlns:xacro="http://www.ros.org/wiki/xacro">
   <xacro:arg name="end_effector_preset" default="dual_motor_gripper"/>

Commit message: feat(arm): XL430 ID1 영점과 결합 잠금 제어 추가

File: extreme-robot/ros2_ws/src/robot_arm_description/urdf/robot_arm.urdf (robot description, URDF)
Before this commit: robot robot_arm, 23 links, 22 joints
Joints:
- joint toolchanger_lock_wheel: limit lower=0 upper=0.392699 effort=10 velocity=2.0 -> effort=10 velocity=2.0; type revolute -> continuous
